File: kicad/picocade.kicad_sch (KiCad schematic)
At the start: 9 parts, among them SW4 SW_Push, U1 PicoW

Commit message: add schematics
Parts:
- added D1: LED, symbol Device:LED
- added R1: 50-330 ohms, symbol Device:R_US
- SW1: renamed from SW_UP; value SW_Push -> SW_Up
- SW2: renamed from SW_DOWN; value SW_Push -> SW_Down
- SW3: renamed from SW_LEFT; value SW_Push -> SW_Left
- SW4: value SW_Push -> SW_Right
- SW5: renamed from SW_F1; value SW_Push -> SW_Esc
- SW6: renamed from SW_F2; value SW_Push -> SW_Splore
- SW7: renamed from SW_Z; value SW_Push -> SW_Z
- SW8: renamed from SW_X; value SW_Push -> SW_X
Connections:
- net GNDREF: now also R1.1
- net at U1.22 (GPIO17): now also D1.2 (A)
- new net: D1.1 (K), R1.2
Other:
- note removed: "0.0.1"
- note removed: "picocade"

Commit message: :baby: fix resistor possition on schematics
Connections:
- net GNDREF: now also D1.1 (K); no longer R1.1
- net at U1.22 (GPIO17): now also R1.2; no longer D1.2 (A)
- new net: D1.2 (A), R1.1
Changed lines of the file:
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@@
-    (stroke (width 0) (type default))
-  )
-  (wire (pts (xy 185.42 130.81) (xy 185.42 132.08))
     (stroke (width 0) (type default))
   )
@@
     (stroke (width 0) (type default))
   )
+  (wire (pts (xy 186.69 90.17) (xy 190.5 90.17))
+    (stroke (width 0) (type default))
+  )
+  (wire (pts (xy 185.42 129.54) (xy 185.42 132.08))
+    (stroke (width 0) (type default))
+  )
+  (wire (pts (xy 127 82.55) (xy 127 102.87))
+    (stroke (width 0) (type default))
+  )
   (wire (pts (xy 172.72 115.57) (xy 185.42 115.57))
     (stroke (width 0) (type default))
   )
-  (wire (pts (xy 186.69 90.17) (xy 190.5 90.17))
-    (stroke (width 0) (type default))
-  )
-  (wire (pts (xy 127 82.55) (xy 127 102.87))
+  (wire (pts (xy 185.42 121.92) (xy 185.42 123.19))
     (stroke (width 0) (type default))
   )
@@
     )
   )
-  (symbol (lib_id "Device:LED") (at 185.42 119.38 90) (unit 1)
-    (in_bom yes) (on_board yes) (dnp no) (fields_autoplaced)
-    (property "Reference" "D1" (at 193.04 120.9675 0)
-      (effects (font (size 1.27 1.27)) hide)
-    )
-    (property "Value" "LED" (at 189.23 120.9675 90)
+  (symbol (lib_id "Device:LED") (at 185.42 125.73 90) (unit 1)
+    (in_bom yes) (on_board yes) (dnp no) (fields_autoplaced)
+    (property "Reference" "D1" (at 193.04 127.3175 0)
+      (effects (font (size 1.27 1.27)) hide)
+    )
+    (property "Value" "LED" (at 189.23 127.3175 90)
       (effects (font (size 1.27 1.27)) (justify right))
     )
-    (property "Footprint" "" (at 185.42 119.38 0)
-      (effects (font (size 1.27 1.27)) hide)
-    )
-    (property "Datasheet" "~" (at 185.42 119.38 0)
+    (property "Footprint" "" (at 185.42 125.73 0)
+      (effects (font (size 1.27 1.27)) hide)
+    )
+    (property "Datasheet" "~" (at 185.42 125.73 0)
       (effects (font (size 1.27 1.27)) hide)
     )
@@
     )
   )
-  (symbol (lib_id "Device:R_US") (at 185.42 127 180) (unit 1)
-    (in_bom yes) (on_board yes) (dnp no) (fields_autoplaced)
-    (property "Reference" "R1" (at 179.07 127 90)
-      (effects (font (size 1.27 1.27)) hide)
-    )
-    (property "Value" "50-330 ohms" (at 187.96 127 0)
+  (symbol (lib_id "Device:R_US") (at 185.42 119.38 180) (unit 1)
+    (in_bom yes) (on_board yes) (dnp no) (fields_autoplaced)
+    (property "Reference" "R1" (at 179.07 119.38 90)
+      (effects (font (size 1.27 1.27)) hide)
+    )
+    (property "Value" "50-330 ohms" (at 187.96 119.38 0)
       (effects (font (size 1.27 1.27)) (justify right))
     )
-    (property "Footprint" "" (at 184.404 126.746 90)
-      (effects (font (size 1.27 1.27)) hide)
-    )
-    (property "Datasheet" "~" (at 185.42 127 0)
-      (effects (font (size 1.27 1.27)) hide)
-    )
+    (property "Footprint" "" (at 184.404 119.126 90)
+      (effects (font (size 1.27 1.27)) hide)
+    )
+    (property "Datasheet" "~" (at 185.42 119.38 0)
+      (effects (font (size 1.27 1.27)) hide)
+    )

Commit message: swap left and right controls
Parts:
- SW3: value SW_Left -> SW_Right
- SW4: value SW_Right -> SW_Left
Changed lines of the file:
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@@
       (effects (font (size 1.27 1.27)) hide)
     )
-    (property "Value" "SW_Right" (at 114.3 97.79 0)
+    (property "Value" "SW_Left" (at 114.3 97.79 0)
       (effects (font (size 1.27 1.27)))
     )
@@
       (effects (font (size 1.27 1.27)) hide)
     )
-    (property "Value" "SW_Left" (at 114.3 85.09 0)
+    (property "Value" "SW_Right" (at 114.3 85.09 0)
       (effects (font (size 1.27 1.27)))
     )
